File: nrf51_1.2/nrf51822.brd (EAGLE design)
At the start: 38.2 x 26.4 mm, 20 parts, among them T1 MMUN2238

Commit message: Sent to smart-prototype Actuation 1.2 Compact 1.1
Changed lines of the file:
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@@
 <layer number="49" name="Reference" color="7" fill="1" visible="yes" active="yes"/>
 <layer number="50" name="dxf" color="7" fill="1" visible="no" active="no"/>
-<layer number="51" name="tDocu" color="13" fill="1" visible="yes" active="yes"/>
+<layer number="51" name="tDocu" color="13" fill="1" visible="no" active="yes"/>
 <layer number="52" name="bDocu" color="7" fill="1" visible="no" active="yes"/>
 <layer number="53" name="tGND_GNDA" color="7" fill="9" visible="no" active="no"/>
@@
 </element>
 <element name="C8" library="rcl" package="C0805" value="100nF" x="17.97" y="19.5" smashed="yes">
-<attribute name="NAME" x="17" y="20.8" size="1.27" layer="25"/>
+<attribute name="NAME" x="15.9586" y="20.7746" size="1.27" layer="25"/>
 </element>
 <element name="C9" library="rcl" package="C0805" value="1.0nF" x="25.166" y="17.8672" smashed="yes">
